Commit message: Making edits to the code so as to remove the kdl error

File: project_orion_description/urdf/orion_vehicle.urdf.xacro (robot description, xacro)
@@ -55,4 +55,11 @@
     </joint>
   </xacro:macro>
+  <!-- ==================== base_footprint (true root, ground level) ==================== -->
+  <link name="base_footprint"/>
+  <joint name="base_footprint_joint" type="fixed">
+    <parent link="base_footprint"/>
+    <child link="base_link"/>
+    <origin xyz="0 0 ${ground_clearance}" rpy="0 0 0"/>
+  </joint>
   <!-- ==================== base_link (chassis) ==================== -->
   <link name="base_link">

Commit message: Testing the rear wheel alone

File: project_orion_description/urdf/orion_vehicle.urdf.xacro (robot description, xacro)
@@ -191,3 +191,36 @@
     <origin xyz="${chassis_length/2} 0 ${camera_size/2}" rpy="0 0 0"/>
   </joint>
+  <ros2_control name="OrionSystem" type="system">
+    <hardware>
+      <plugin>mock_components/GenericSystem</plugin>
+    </hardware>
+    <joint name="rear_left_wheel_joint">
+      <command_interface name="velocity"/>
+      <state_interface name="velocity"/>
+      <state_interface name="position"/>
+    </joint>
+    <joint name="rear_right_wheel_joint">
+      <command_interface name="velocity"/>
+      <state_interface name="velocity"/>
+      <state_interface name="position"/>
+    </joint>
+    <joint name= "front_left_wheel_joint">
+      <command_interface name="velocity"/>
+      <state_interface name="position"/>
+      <state_interface name="velocity"/>
+    </joint>
+    <joint name= "front_right_wheel_joint"/>
+      <command_interface name="velocity"/>
+      <state_interface name="velocity"/>
+      <state_interface name="position"/>
+    <joint>
+    <joint name = "front_left_steering_joint"/>
+      <command_interface name="velocity"/>
+      <state_interface nsme="position"/>
+    </joint>
+    <joint name = "front_right_steering_joint">
+      <command_interface name= "velocity"/>
+      <state_interface name="position"/>
+    </joint>
+  </ros2_control>
 </robot>

Commit message: docs: Stage4/5 writeup , debugging logs, physics reference

File: project_orion_description/urdf/orion_vehicle.urdf.xacro (robot description, xacro)
@@ -15,4 +15,5 @@
   <!-- Ground clearance: distance from ground to base_link origin -->
   <xacro:property name="ground_clearance" value="${wheel_radius}"/>
+  <xacro:arg name="use_mock" default="true"/>
   <!-- ==================== Materials ==================== -->
   <material name="orion_body_color">
@@ -193,5 +194,10 @@
   <ros2_control name="OrionSystem" type="system">
     <hardware>
-      <plugin>mock_components/GenericSystem</plugin>
+      <xacro:if value="$(arg use_mock)">
+        <plugin>mock_components/GenericSystem</plugin>
+      </xacro:if>
+      <xacro:unless value="$(arg use_mock)">
+        <plugin>gz_ros2_control/GazeboSimSystem</plugin>
+      </xacro:unless>
     </hardware>
     <joint name="rear_left_wheel_joint">
@@ -205,20 +211,20 @@
       <state_interface name="position"/>
     </joint>
-    <joint name= "front_left_wheel_joint">
-      <command_interface name="velocity"/>
-      <state_interface name="position"/>
-      <state_interface name="velocity"/>
-    </joint>
-    <joint name= "front_right_wheel_joint"/>
-      <command_interface name="velocity"/>
-      <state_interface name="velocity"/>
-      <state_interface name="position"/>
-    <joint>
-    <joint name = "front_left_steering_joint"/>
-      <command_interface name="velocity"/>
-      <state_interface nsme="position"/>
-    </joint>
-    <joint name = "front_right_steering_joint">
-      <command_interface name= "velocity"/>
+    <joint name="front_left_wheel_joint">
+      <command_interface name="velocity"/>
+      <state_interface name="position"/>
+      <state_interface name="velocity"/>
+    </joint>
+    <joint name="front_right_wheel_joint">
+      <command_interface name="velocity"/>
+      <state_interface name="velocity"/>
+      <state_interface name="position"/>
+    </joint>
+    <joint name="front_left_steering_joint">
+      <command_interface name="position"/>
+      <state_interface name="position"/>
+    </joint>
+    <joint name="front_right_steering_joint">
+      <command_interface name="position"/>
       <state_interface name="position"/>
     </joint>

File: project_orion_simulation/urdf/orion_vehicle.gazebo.xacro (robot description, xacro)
@@ -2,4 +2,9 @@
 <robot name="orion_vehicle" xmlns:xacro="http://www.ros.org/wiki/xacro">
   <xacro:include filename="$(find project_orion_description)/urdf/orion_vehicle.urdf.xacro"/>
+  <gazebo>
+    <plugin filename="gz_ros2_control-system" name="gz_ros2_control::GazeboSimROS2ControlPlugin">
+      <parameters>$(find project_orion_control)/config/orion_controllers.yaml</parameters>
+    </plugin>
+  </gazebo>
   <gazebo reference="base_link">
     <material>Gazebo/Blue</material>
